Commit message: Добавлен пакет slam_with_filter и изменены файлы модели робота

File: src/two_wheeled_robot/install/two_wheeled_robot/share/two_wheeled_robot/urdf/two_wheeled_robot.urdf (robot description, URDF)
Before this commit: robot two_wheeled_robot, 6 links, 5 joints
Joints:
- joint camera_joint: axis (none) -> 0 0 1; limit (none) -> effort=1000 velocity=10; type fixed -> continuous

File: src/two_wheeled_robot/install/two_wheeled_robot/share/two_wheeled_robot/urdf/two_wheeled_robot_with_gazebo_plugins.urdf (robot description, URDF)
Before this commit: robot two_wheeled_robot, 6 links, 5 joints
Joints:
- joint camera_joint: axis (none) -> 0 0 1; type fixed -> continuous

File: src/two_wheeled_robot/urdf/two_wheeled_robot.urdf (robot description, URDF)
Before this commit: robot two_wheeled_robot, 6 links, 5 joints
Joints:
- joint camera_joint: axis (none) -> 0 0 1; type fixed -> continuous

File: src/two_wheeled_robot/urdf/two_wheeled_robot_with_gazebo_plugins.urdf (robot description, URDF)
Before this commit: robot two_wheeled_robot, 6 links, 5 joints
Joints:
- joint camera_joint: axis (none) -> 0 0 1; type fixed -> continuous
